File: PCB/ServoTesterBoard/ServoTesterBoard.kicad_pcb (KiCad board)
At the start: 2 copper layers, 70.5 x 41.1 mm, 23 parts, among them J1 Barrel Jack, J2 2.54mm 1x2 Header, J3 2.54mm 1x3 Header, Q1 BC547, SW1 Slide Switch, SW2 Push Button, SW3 Push Button, U1 LM555xM, U2 L7805

Commit message: Finished
Parts:
- added R7: 470, Resistor_SMD:R_1206_3216Metric_Pad1.30x1.75mm_HandSolder, F.Cu at (182.2, 72.0)
- moved C2 0.75 mm to (171.5, 76.1)
- moved C4 0.75 mm to (178.5, 74.0)
Routing:
- net /ServoData: track 24.3 -> 26.5 mm
- net 5V0: track 102.5 -> 101.9 mm
- added copper zone on B.Cu, net GND
Other:
- board text added: "Nicholas Niles"
- board text removed: "Nicholas Niles 24'"
- board text removed: "in 26'"
